File: hardware/kicad/v1_0/arduino_nano_reflow_TRIAC_v1_0.sch (KiCad schematic (older format))
At the start: 34 parts, among them J1 AC IN 220v, J10 CONN_01X17, J11 CONN_01X03, J12 MOUNTING_HOLE, J13 MOUNTING_HOLE, J14 MOUNTING_HOLE, J15 MOUNTING_HOLE, J2 HEATER, J3 DC IN 12V, J4 12v FAN, J5 CONN_01X03, J6 CONN_01X03, J7 CONN_01X03, J8 CONN_01X03, J9 CONN_01X05, Q1 IRF540N, U1 MOC3020M

Commit message: - new revision of board - suitable for production with oshpark - updated footprints - cross checked with original schematics
Parts:
- BZ1: footprint Buzzers_Beepers:Buzzer_12x9.5RM7.6 -> Buzzer_Beeper:Buzzer_12x9.5RM7.6
- C2: footprint Capacitors_SMD:C_0805 -> Capacitor_SMD:C_0805_2012Metric
- J12, J13, J14, J15: footprint Mounting_Holes:MountingHole_3.2mm_M3_Pad_Via -> MountingHole:MountingHole_3.2mm_M3_Pad
- Q1: footprint TO_SOT_Packages_THT:TO-220_Vertical -> Package_TO_SOT_THT:TO-220-3_Vertical; symbol arduino_nano_reflow_TRIAC_v1_0-rescue:IRF540N -> Transistor_FET:IRF540N
- R1, R2: footprint Resistors_THT:R_Axial_DIN0207_L6.3mm_D2.5mm_P7.62mm_Horizontal -> Resistor_THT:R_Axial_DIN0207_L6.3mm_D2.5mm_P7.62mm_Horizontal
- R6, R7: footprint Resistors_SMD:R_1210 -> Resistor_SMD:R_1210_3225Metric
Connections:
- net labels removed: 3V3, AC2
- wire segments 84 -> 90
- no-connect marks 10 -> 7
Other:
- moved on the sheet: Q1
Changed lines of the file:
@@
 F 0 "C2" H 3800 4150 70  0000 L BNN
 F 1 "100n" H 3800 3950 70  0000 L BNN
-F 2 "Capacitors_SMD:C_0805" H 3740 3890 65  0001 L TNN
+F 2 "Capacitor_SMD:C_0805_2012Metric" H 3740 3890 65  0001 L TNN
 F 3 "" H 3750 4100 60  0001 C CNN
 	1    3750 4100
@@
 F 0 "R2" V 3150 1650 70  0000 L BNN
 F 1 "47k 0.6w" V 3050 1650 70  0000 L BNN
-F 2 "Resistors_THT:R_Axial_DIN0207_L6.3mm_D2.5mm_P7.62mm_Horizontal" H 2890 1540 65  0001 L TNN
+F 2 "Resistor_THT:R_Axial_DIN0207_L6.3mm_D2.5mm_P7.62mm_Horizontal" H 2890 1540 65  0001 L TNN
 F 3 "" H 2900 1750 60  0001 C CNN
 	1    2900 1750
@@
 F 0 "R7" H 6430 3870 50  0000 L CNN
 F 1 "100K" H 6430 3810 50  0000 L CNN
-F 2 "Resistors_SMD:R_1210" H 6400 3850 50  0001 C CNN
+F 2 "Resistor_SMD:R_1210_3225Metric" H 6400 3850 50  0001 C CNN
 F 3 "" H 6400 3850 50  0001 C CNN
 	1    6400 3850
@@
 D6
 $Comp
-L arduino_nano_reflow_TRIAC_v1_0-rescue:IRF540N Q1
+L Transistor_FET:IRF540N Q1
 U 1 1 5922ADDA
-P 6750 4200
-F 0 "Q1" H 6950 4000 50  0000 L CNN
-F 1 "IRF540N" H 6950 4100 50  0000 L CNN
-F 2 "TO_SOT_Packages_THT:TO-220_Vertical" H 7000 4125 50  0001 L CIN
-F 3 "" H 6750 4200 50  0001 L CNN
-	1    6750 4200
+P 6750 4150
+F 0 "Q1" H 6950 3950 50  0000 L CNN
+F 1 "IRF540N" H 6950 4050 50  0000 L CNN
+F 2 "Package_TO_SOT_THT:TO-220-3_Vertical" H 7000 4075 50  0001 L CIN
+F 3 "http://www.irf.com/product-info/datasheets/data/irf540n.pdf" H 6750 4150 50  0001 L CNN
+	1    6750 4150
 	1    0    0    1
 $EndComp
@@
 F 0 "BZ1" H 4250 4600 50  0000 L CNN
 F 1 "Buzzer" H 4250 4500 50  0000 L CNN
-F 2 "Buzzers_Beepers:Buzzer_12x9.5RM7.6" V 4075 4650 50  0001 C CNN
+F 2 "Buzzer_Beeper:Buzzer_12x9.5RM7.6" V 4075 4650 50  0001 C CNN
 F 3 "" V 4075 4650 50  0001 C CNN
 	1    4100 4550
@@
 F 0 "R6" V 6050 4150 50  0000 L CNN
 F 1 "4K7" V 5950 4100 50  0000 L CNN
-F 2 "Resistors_SMD:R_1210" H 6150 4150 50  0001 C CNN
+F 2 "Resistor_SMD:R_1210_3225Metric" H 6150 4150 50  0001 C CNN
 F 3 "" H 6150 4150 50  0001 C CNN
 	1    6150 4150
@@
 Text GLabel 10000 2950 2    60   Input ~ 0
 GND
-Text Label 3200 5150 0    47   ~ 0
-3V3
 Text GLabel 9800 2400 2    60   Input ~ 0
 5V
@@
 F 0 "J15" H 2650 7050 50  0000 C CNN
 F 1 "MOUNTING_HOLE" H 3100 6950 50  0000 C CNN
-F 2 "Mounting_Holes:MountingHole_3.2mm_M3_Pad_Via" H 2650 6950 50  0001 C CNN
+F 2 "MountingHole:MountingHole_3.2mm_M3_Pad" H 2650 6950 50  0001 C CNN
 F 3 "" H 2650 6950 50  0001 C CNN
 	1    2650 6950
@@
 F 0 "J12" H 1900 6700 50  0000 C CNN
 F 1 "MOUNTING_HOLE" H 2350 6600 50  0000 C CNN
-F 2 "Mounting_Holes:MountingHole_3.2mm_M3_Pad_Via" H 1900 6600 50  0001 C CNN
+F 2 "MountingHole:MountingHole_3.2mm_M3_Pad" H 1900 6600 50  0001 C CNN
 F 3 "" H 1900 6600 50  0001 C CNN
 	1    1900 6600
 	-1   0    0    -1
 $EndComp
-NoConn ~ 2100 6600
 $Comp
 L arduino_nano_reflow_TRIAC_v1_0-rescue:CONN_01X01 J13
@@
 F 0 "J13" H 1900 7050 50  0000 C CNN
 F 1 "MOUNTING_HOLE" H 2350 6950 50  0000 C CNN
-F 2 "Mounting_Holes:MountingHole_3.2mm_M3_Pad_Via" H 1900 6950 50  0001 C CNN
+F 2 "MountingHole:MountingHole_3.2mm_M3_Pad" H 1900 6950 50  0001 C CNN
 F 3 "" H 1900 6950 50  0001 C CNN
 	1    1900 6950
 	-1   0    0    -1
 $EndComp
-NoConn ~ 2100 6950
 Text GLabel 6900 2350 2    60   Input ~ 0
 GND
@@
 Text Label 5000 1750 0    39   ~ 0
 AC_CAP
-NoConn ~ 2450 6950
 Text Label 2550 2050 0    39   ~ 0
 OC2
@@
 F 0 "J14" H 2650 6700 50  0000 C CNN
 F 1 "MOUNTING_HOLE" H 3100 6600 50  0000 C CNN
-F 2 "Mounting_Holes:MountingHole_3.2mm_M3_Pad_Via" H 2650 6600 50  0001 C CNN
+F 2 "MountingHole:MountingHole_3.2mm_M3_Pad" H 2650 6600 50  0001 C CNN
 F 3 "" H 2650 6600 50  0001 C CNN
 	1    2650 6600
 	1    0    0    -1
 $EndComp
-NoConn ~ 2450 6600
 Text Label 8750 2550 0    47   ~ 0
 ENC_1
@@
 F 0 "R1" V 2850 1950 70  0000 L BNN
 F 1 "47k 0.6w" V 2750 1950 70  0000 L BNN
-F 2 "Resistors_THT:R_Axial_DIN0207_L6.3mm_D2.5mm_P7.62mm_Horizontal" H 2890 1840 65  0001 L TNN
+F 2 "Resistor_THT:R_Axial_DIN0207_L6.3mm_D2.5mm_P7.62mm_Horizontal" H 2890 1840 65  0001 L TNN
 F 3 "" H 2900 2050 60  0001 C CNN
 	1    2900 2050
@@
 	3200 4150 3350 4150
 Wire Wire Line
-	6850 3550 6850 4000
+	6850 3550 6850 3950
 Wire Wire Line
 	6400 3750 6400 3550
@@
 	6400 3950 6400 4150
 Connection ~ 6400 4150
-Wire Wire Line
-	6850 4400 6850 4700
 Wire Wire Line
 	2100 4150 2200 4150
@@
 AC1_OUT
 Text GLabel 3150 2050 2    60   Input ~ 0
-AC2
+AC2_IN
 Text GLabel 3150 1750 2    60   Input ~ 0
 AC1_IN
@@
 	3200 3950 3750 3950
 Connection ~ 3750 3950
+Text GLabel 2275 7000 3    60   Input ~ 0
+GND
+Wire Wire Line
+	2100 6600 2275 6600
+Wire Wire Line
+	2275 6600 2275 6950
+Wire Wire Line
+	2100 6950 2275 6950
+Connection ~ 2275 6950
+Wire Wire Line
+	2275 6950 2275 7000
+Wire Wire Line
+	2450 6950 2275 6950
+Wire Wire Line
+	2450 6600 2275 6600
+Connection ~ 2275 6600
+Wire Wire Line
+	6850 4350 6850 4700
+NoConn ~ 3200 5150
 $EndSCHEMATC

Commit message: update footprint to match kicad 5.1.6 - SIP suitable for oshpark
Parts:
- ARDUINO_NANO1: footprint local_modules:arduino_nano_header -> Module:Arduino_Nano
- C1: footprint Capacitors_THT:C_Disc_D4.3mm_W1.9mm_P5.00mm -> Capacitor_THT:C_Disc_D4.3mm_W1.9mm_P5.00mm
- D1: footprint Diodes_THT:D_A-405_P5.08mm_Vertical_AnodeUp -> Diode_THT:D_A-405_P5.08mm_Vertical_AnodeUp
- J1, J2, J3: footprint Connectors_Terminal_Blocks:TerminalBlock_Pheonix_MKDS1.5-2pol -> TerminalBlock_Phoenix:TerminalBlock_Phoenix_MKDS-1,5-2_1x02_P5.00mm_Horizontal
- J10: footprint Pin_Headers:Pin_Header_Straight_1x17_Pitch2.54mm -> Connector_PinHeader_2.54mm:PinHeader_1x17_P2.54mm_Vertical; symbol arduino_nano_reflow_TRIAC_v1_0-rescue:CONN_01X17 -> Connector_Generic:Conn_01x17
- J9: footprint Pin_Headers:Pin_Header_Straight_1x05_Pitch2.54mm -> Connector_PinHeader_2.54mm:PinHeader_1x05_P2.54mm_Vertical; symbol arduino_nano_reflow_TRIAC_v1_0-rescue:CONN_01X05 -> Connector_Generic:Conn_01x05
- OK1: footprint Housings_DIP:DIP-6_W7.62mm_LongPads -> Package_DIP:DIP-6_W7.62mm; symbol H11AA1:H11AA1 -> Isolator:H11AA1
- R3, R4: footprint Resistors_THT:R_Axial_DIN0207_L6.3mm_D2.5mm_P7.62mm_Horizontal -> Resistor_THT:R_Axial_DIN0207_L6.3mm_D2.5mm_P7.62mm_Horizontal
- R5: footprint Resistors_SMD:R_0603 -> Resistor_SMD:R_0603_1608Metric
- TRIAC1: footprint local_modules:TO-220_Vertical_BT137 -> Package_TO_SOT_THT:TO-220-3_Vertical; symbol BT137:BT137 -> Device:Q_TRIAC_A1A2G
- U1: footprint Housings_DIP:DIP-6_W7.62mm_LongPads -> Package_DIP:DIP-6_W7.62mm; symbol arduino_nano_reflow_TRIAC_v1_0-rescue:MOC3020M -> Relay_SolidState:MOC3020M
Connections:
- wire segments 90 -> 96
Changed lines of the file:
@@
 F 0 "ARDUINO_NANO1" H 2850 5350 60  0000 C CNN
 F 1 "arduino_nano_header" H 2850 3750 60  0000 C CNN
-F 2 "local_modules:arduino_nano_header" H 2850 3600 60  0001 C CNN
+F 2 "Module:Arduino_Nano" H 2850 3600 60  0001 C CNN
 F 3 "" H 2850 4550 60  0000 C CNN
 	1    2850 4550
@@
 F 0 "J2" H 5100 7350 50  0000 C TNN
 F 1 "HEATER" V 4950 7100 50  0000 C TNN
-F 2 "Connectors_Terminal_Blocks:TerminalBlock_Pheonix_MKDS1.5-2pol" H 5100 6875 50  0001 C CNN
+F 2 "TerminalBlock_Phoenix:TerminalBlock_Phoenix_MKDS-1,5-2_1x02_P5.00mm_Horizontal" H 5100 6875 50  0001 C CNN
 F 3 "" H 5075 7100 50  0001 C CNN
 	1    5100 7100
@@
 F 0 "J3" H 5750 7350 50  0000 C TNN
 F 1 "DC IN 12V" V 5600 7100 50  0000 C TNN
-F 2 "Connectors_Terminal_Blocks:TerminalBlock_Pheonix_MKDS1.5-2pol" H 5750 6875 50  0001 C CNN
+F 2 "TerminalBlock_Phoenix:TerminalBlock_Phoenix_MKDS-1,5-2_1x02_P5.00mm_Horizontal" H 5750 6875 50  0001 C CNN
 F 3 "" H 5725 7100 50  0001 C CNN
 	1    5750 7100
@@
 F 0 "J1" H 4450 7350 50  0000 C TNN
 F 1 "AC IN 220v" V 4300 7100 50  0000 C TNN
-F 2 "Connectors_Terminal_Blocks:TerminalBlock_Pheonix_MKDS1.5-2pol" H 4450 6875 50  0001 C CNN
+F 2 "TerminalBlock_Phoenix:TerminalBlock_Phoenix_MKDS-1,5-2_1x02_P5.00mm_Horizontal" H 4450 6875 50  0001 C CNN
 F 3 "" H 4425 7100 50  0001 C CNN
 	1    4450 7100
@@
 F 0 "D1" H 6950 4780 50  0000 L CNN
 F 1 "1N4007" H 6850 4620 50  0000 L CNN
-F 2 "Diodes_THT:D_A-405_P5.08mm_Vertical_AnodeUp" V 7000 4700 50  0001 C CNN
+F 2 "Diode_THT:D_A-405_P5.08mm_Vertical_AnodeUp" V 7000 4700 50  0001 C CNN
 F 3 "" V 7000 4700 50  0001 C CNN
 	1    7000 4700
@@
 FAN_CTRL
 $Comp
-L arduino_nano_reflow_TRIAC_v1_0-rescue:CONN_01X05 J9
+L Connector_Generic:Conn_01x05 J9
 U 1 1 592EA702
 P 9600 2300
 F 0 "J9" H 9600 2600 50  0000 C CNN
 F 1 "CONN_01X05" V 9700 2300 50  0000 C CNN
-F 2 "Pin_Headers:Pin_Header_Straight_1x05_Pitch2.54mm" H 9600 2300 50  0001 C CNN
+F 2 "Connector_PinHeader_2.54mm:PinHeader_1x05_P2.54mm_Vertical" H 9600 2300 50  0001 C CNN
 F 3 "" H 9600 2300 50  0001 C CNN
 	1    9600 2300
@@
 VIN
 $Comp
-L arduino_nano_reflow_TRIAC_v1_0-rescue:CONN_01X17 J10
+L Connector_Generic:Conn_01x17 J10
 U 1 1 592F1E66
 P 9600 3750
 F 0 "J10" H 9600 4650 50  0000 C CNN
 F 1 "CONN_01X17" V 9700 3750 50  0000 C CNN
-F 2 "Pin_Headers:Pin_Header_Straight_1x17_Pitch2.54mm" H 9600 3750 50  0001 C CNN
+F 2 "Connector_PinHeader_2.54mm:PinHeader_1x17_P2.54mm_Vertical" H 9600 3750 50  0001 C CNN
 F 3 "" H 9600 3750 50  0001 C CNN
 	1    9600 3750
@@
 F 0 "R5" V 6800 2250 70  0000 R TNN
 F 1 "1k" V 6700 2250 70  0000 R TNN
-F 2 "Resistors_SMD:R_0603" H 6640 1940 65  0001 L TNN
+F 2 "Resistor_SMD:R_0603_1608Metric" H 6640 1940 65  0001 L TNN
 F 3 "" H 6650 2150 60  0001 C CNN
 	1    6650 2150
@@
 F 0 "R3" V 5050 1650 70  0000 L BNN
 F 1 "2.4k" V 4950 1650 70  0000 L BNN
-F 2 "Resistors_THT:R_Axial_DIN0207_L6.3mm_D2.5mm_P7.62mm_Horizontal" H 4790 1540 65  0001 L TNN
+F 2 "Resistor_THT:R_Axial_DIN0207_L6.3mm_D2.5mm_P7.62mm_Horizontal" H 4790 1540 65  0001 L TNN
 F 3 "" H 4800 1750 60  0001 C CNN
 	1    4800 1750
@@
 GND
 $Comp
-L arduino_nano_reflow_TRIAC_v1_0-rescue:MOC3020M U1
+L Relay_SolidState:MOC3020M U1
 U 1 1 594CBE26
 P 6050 2250
 F 0 "U1" H 5840 2440 50  0000 L CNN
 F 1 "MOC3020M" H 5850 2550 50  0000 L CNN
-F 2 "Housings_DIP:DIP-6_W7.62mm_LongPads" H 5850 2050 50  0001 L CIN
-F 3 "" H 6025 2250 50  0001 L CNN
+F 2 "Package_DIP:DIP-6_W7.62mm" H 5850 2050 50  0001 L CIN
+F 3 "http://www.fairchildsemi.com/ds/MO/MOC3020M.pdf" H 6025 2250 50  0001 L CNN
 	1    6050 2250
 	-1   0    0    -1
@@
 F 0 "R4" V 5700 1650 70  0000 L BNN
 F 1 "180R" V 5600 1650 70  0000 L BNN
-F 2 "Resistors_THT:R_Axial_DIN0207_L6.3mm_D2.5mm_P7.62mm_Horizontal" H 5440 1540 65  0001 L TNN
+F 2 "Resistor_THT:R_Axial_DIN0207_L6.3mm_D2.5mm_P7.62mm_Horizontal" H 5440 1540 65  0001 L TNN
 F 3 "" H 5450 1750 60  0001 C CNN
 	1    5450 1750
@@
 F 0 "C1" H 4900 1950 70  0000 L BNN
 F 1 "10n" H 4850 2050 70  0000 L BNN
-F 2 "Capacitors_THT:C_Disc_D4.3mm_W1.9mm_P5.00mm" H 5140 1840 65  0001 L TNN
+F 2 "Capacitor_THT:C_Disc_D4.3mm_W1.9mm_P5.00mm" H 5140 1840 65  0001 L TNN
 F 3 "" H 5150 2050 60  0001 C CNN
 	1    5150 2050
@@
 $EndComp
 $Comp
-L H11AA1:H11AA1 OK1
+L Isolator:H11AA1 OK1
 U 1 1 594F8B28
 P 2000 1850
 F 0 "OK1" H 2050 2100 45  0000 L BNN
 F 1 "H11AA1" H 1950 1450 45  0000 L BNN
-F 2 "Housings_DIP:DIP-6_W7.62mm_LongPads" H 2030 2000 20  0001 C CNN
-F 3 "" H 2000 1850 60  0001 C CNN
+F 2 "Package_DIP:DIP-6_W7.62mm" H 2030 2000 20  0001 C CNN
+F 3 "https://www.vishay.com/docs/83608/h11aa1.pdf" H 2000 1850 60  0001 C CNN
 	1    2000 1850
 	-1   0    0    -1
 $EndComp
 $Comp
-L BT137:BT137 TRIAC1
+L Device:Q_TRIAC_A1A2G TRIAC1
 U 1 1 594F8C53
 P 4500 2250
 F 0 "TRIAC1" H 4625 2275 50  0000 L CNN
 F 1 "BT137" H 4625 2200 50  0000 L CNN
-F 2 "local_modules:TO-220_Vertical_BT137" V 4575 2275 50  0001 C CNN
+F 2 "Package_TO_SOT_THT:TO-220-3_Vertical" V 4575 2275 50  0001 C CNN
 F 3 "" V 4500 2250 50  0001 C CNN
 	1    4500 2250
-	-1   0    0    -1
+	1    0    0    -1
 $EndComp
 Text Label 3200 4450 0    47   ~ 0
@@
 Wire Wire Line
 	5750 2150 5750 1750
-Wire Wire Line
-	5750 2350 4650 2350
 Connection ~ 5150 1750
 Wire Wire Line
@@
 Text GLabel 3150 1750 2    60   Input ~ 0
 AC1_IN
-Wire Wire Line
-	2750 1750 2550 1750
-Wire Wire Line
-	2750 2050 2550 2050
 Text GLabel 4400 1750 0    60   Input ~ 0
 AC1_IN
@@
 	6850 4350 6850 4700
 NoConn ~ 3200 5150
+Wire Wire Line
+	5750 2350 5300 2350
+Wire Wire Line
+	5300 2350 5300 2750
+Wire Wire Line
+	5300 2750 3900 2750
+Wire Wire Line
+	3900 2750 3900 2350
+Wire Wire Line
+	3900 2350 4350 2350
+Wire Wire Line
+	1700 1950 1700 2050
+Wire Wire Line
+	2300 1750 2750 1750
+Wire Wire Line
+	2300 1950 2300 2050
+Wire Wire Line
+	2300 2050 2750 2050
 $EndSCHEMATC

Commit message: updated PCB to v1.0_rev3 - more space for connectors and rewired for better access to FAN port
Parts:
- removed J4: 12v FAN, Pin_Headers:Pin_Header_Straight_2x01_Pitch2.54mm, symbol arduino_nano_reflow_TRIAC_v1_0-rescue:CONN_01X02
- removed J5, J6, J7, J8: CONN_01X03, Pin_Headers:Pin_Header_Straight_1x03_Pitch2.54mm, symbol arduino_nano_reflow_TRIAC_v1_0-rescue:CONN_01X03
- added J4: 12V FAN, TerminalBlock_Phoenix:TerminalBlock_Phoenix_MKDS-1,5-2_1x02_P5.00mm_Horizontal, symbol arduino_nano_reflow_TRIAC_v1_0-rescue:Screw_Terminal_1x02
- BZ1: value Buzzer -> Buzzer with generator
- JP1: symbol Device:Jumper -> Jumper:Jumper_2_Open
- renumbered ARDUINO_NANO1 to ARDUINO_NANO_(5V)1
Connections:
- net 12v: now also J4.2
- net FAN_GND: now also J4.1
Changed lines of the file:
@@
 NoConn ~ 3200 5050
 $Comp
-L arduino-headers:arduino_nano_header ARDUINO_NANO1
+L arduino-headers:arduino_nano_header ARDUINO_NANO_(5V)1
 U 1 1 58EC872C
 P 2850 4550
-F 0 "ARDUINO_NANO1" H 2850 5350 60  0000 C CNN
+F 0 "ARDUINO_NANO_(5V)1" H 2850 5350 60  0000 C CNN
 F 1 "arduino_nano_header" H 2850 3750 60  0000 C CNN
 F 2 "Module:Arduino_Nano" H 2850 3600 60  0001 C CNN
@@
 U 1 1 591B0993
 P 3750 4100
-F 0 "C2" H 3800 4150 70  0000 L BNN
-F 1 "100n" H 3800 3950 70  0000 L BNN
+F 0 "C2" H 3875 4125 70  0000 L BNN
+F 1 "100n" H 3875 4025 70  0000 L BNN
 F 2 "Capacitor_SMD:C_0805_2012Metric" H 3740 3890 65  0001 L TNN
 F 3 "" H 3750 4100 60  0001 C CNN
@@
 P 4100 4550
 F 0 "BZ1" H 4250 4600 50  0000 L CNN
-F 1 "Buzzer" H 4250 4500 50  0000 L CNN
+F 1 "Buzzer with generator" H 4250 4500 50  0000 L CNN
 F 2 "Buzzer_Beeper:Buzzer_12x9.5RM7.6" V 4075 4650 50  0001 C CNN
 F 3 "" V 4075 4650 50  0001 C CNN
@@
 Text Label 3200 4550 0    47   ~ 0
 A4
-Text GLabel 8500 3650 2    60   Input ~ 0
-GND
-Text GLabel 8500 3550 2    60   Input ~ 0
-GND
-Text GLabel 8500 3450 2    60   Input ~ 0
-GND
-Text GLabel 8500 2900 2    60   Input ~ 0
-5V
-Text GLabel 8500 3000 2    60   Input ~ 0
-5V
-Text GLabel 8500 3100 2    60   Input ~ 0
-5V
-Text GLabel 8500 4200 2    60   Input ~ 0
-12v
-Text GLabel 8500 4100 2    60   Input ~ 0
-12v
-Text GLabel 8500 4000 2    60   Input ~ 0
-12v
-$Comp
-L Device:Jumper JP1
+$Comp
+L Jumper:Jumper_2_Open JP1
 U 1 1 592F07D7
 P 3700 3850
@@
 Text GLabel 9800 2400 2    60   Input ~ 0
 5V
-$Comp
-L arduino_nano_reflow_TRIAC_v1_0-rescue:CONN_01X03 J5
-U 1 1 5932D012
-P 8300 2450
-F 0 "J5" H 8300 2650 50  0000 C CNN
-F 1 "CONN_01X03" V 8400 2450 50  0000 C CNN
-F 2 "Pin_Headers:Pin_Header_Straight_1x03_Pitch2.54mm" H 8300 2450 50  0001 C CNN
-F 3 "" H 8300 2450 50  0001 C CNN
-	1    8300 2450
-	-1   0    0    1
-$EndComp
-$Comp
-L arduino_nano_reflow_TRIAC_v1_0-rescue:CONN_01X03 J6
-U 1 1 5932D24B
-P 8300 3000
-F 0 "J6" H 8300 3200 50  0000 C CNN
-F 1 "CONN_01X03" V 8400 3000 50  0000 C CNN
-F 2 "Pin_Headers:Pin_Header_Straight_1x03_Pitch2.54mm" H 8300 3000 50  0001 C CNN
-F 3 "" H 8300 3000 50  0001 C CNN
-	1    8300 3000
-	-1   0    0    1
-$EndComp
-$Comp
-L arduino_nano_reflow_TRIAC_v1_0-rescue:CONN_01X03 J7
-U 1 1 5932D3FD
-P 8300 3550
-F 0 "J7" H 8300 3750 50  0000 C CNN
-F 1 "CONN_01X03" V 8400 3550 50  0000 C CNN
-F 2 "Pin_Headers:Pin_Header_Straight_1x03_Pitch2.54mm" H 8300 3550 50  0001 C CNN
-F 3 "" H 8300 3550 50  0001 C CNN
-	1    8300 3550
-	-1   0    0    1
-$EndComp
-$Comp
-L arduino_nano_reflow_TRIAC_v1_0-rescue:CONN_01X03 J8
-U 1 1 5932D690
-P 8300 4100
-F 0 "J8" H 8300 4300 50  0000 C CNN
-F 1 "CONN_01X03" V 8400 4100 50  0000 C CNN
-F 2 "Pin_Headers:Pin_Header_Straight_1x03_Pitch2.54mm" H 8300 4100 50  0001 C CNN
-F 3 "" H 8300 4100 50  0001 C CNN
-	1    8300 4100
-	-1   0    0    1
-$EndComp
 Text GLabel 1550 2050 0    60   Input ~ 0
 GND
-$Comp
-L arduino_nano_reflow_TRIAC_v1_0-rescue:CONN_01X02 J4
-U 1 1 5932F8DA
-P 7000 5350
-F 0 "J4" H 7000 5500 50  0000 C CNN
-F 1 "12v FAN" V 7100 5350 50  0000 C CNN
-F 2 "Pin_Headers:Pin_Header_Straight_2x01_Pitch2.54mm" H 7000 5350 50  0001 C CNN
-F 3 "" H 7000 5350 50  0001 C CNN
-	1    7000 5350
-	0    -1   1    0
-$EndComp
 $Comp
 L Device:R R5
@@
 	1    0    0    -1
 $EndComp
-Text Label 8750 2550 0    47   ~ 0
-ENC_1
-Text Label 8750 2450 0    47   ~ 0
-ENC_2
-Text Label 8750 2350 0    47   ~ 0
-ENC_3
 $Comp
 L arduino_nano_reflow_TRIAC_v1_0-rescue:CONN_01X03 J11
@@
 Text Label 2350 4650 2    47   ~ 0
 D6
-Text Label 8500 2350 0    47   ~ 0
-A2
-Text Label 8500 2450 0    47   ~ 0
-A3
-Text Label 8500 2550 0    47   ~ 0
-A4
-Wire Wire Line
-	8500 2550 8750 2550
-Wire Wire Line
-	8750 2450 8500 2450
-Wire Wire Line
-	8500 2350 8750 2350
 Wire Notes Line
 	5300 5650 5300 3400
@@
 	6900 2150 6800 2150
 Wire Wire Line
-	7150 5150 7050 5150
-Wire Wire Line
-	6850 5150 6950 5150
+	7150 5150 7100 5150
+Wire Wire Line
+	6850 5150 6900 5150
 Wire Wire Line
 	10000 2950 9800 2950
@@
 Wire Wire Line
 	9800 4250 9800 4350
-Wire Wire Line
-	4100 3850 4000 3850
 Wire Wire Line
 	1550 2050 1700 2050
@@
 Wire Wire Line
 	7150 4500 7150 4700
-Wire Wire Line
-	3200 3850 3400 3850
 Wire Wire Line
 	3200 4150 3350 4150
@@
 Wire Wire Line
 	2300 2050 2750 2050
+Wire Wire Line
+	3200 3850 3500 3850
+Wire Wire Line
+	3900 3850 4100 3850
+$Comp
+L arduino_nano_reflow_TRIAC_v1_0-rescue:Screw_Terminal_1x02 J4
+U 1 1 5F64DEBD
+P 7000 5350
+F 0 "J4" H 7000 5600 50  0000 C TNN
+F 1 "12V FAN" V 6850 5350 50  0000 C TNN
+F 2 "TerminalBlock_Phoenix:TerminalBlock_Phoenix_MKDS-1,5-2_1x02_P5.00mm_Horizontal" H 7000 5125 50  0001 C CNN
+F 3 "" H 6975 5350 50  0001 C CNN
+	1    7000 5350
+	0    -1   -1   0
+$EndComp
 $EndSCHEMATC

Commit message: add missing heatsink footprint
Parts:
- KK1: footprint local_modules:SK_09_20_SA_TO_220 -> local_libraries:TO_220_heatsink
Changed lines of the file:
@@
 F 0 "KK1" H 6200 1300 45  0000 L BNN
 F 1 "TRIAC HEATSINK" H 6200 1200 45  0000 L BNN
-F 2 "local_modules:SK_09_20_SA_TO_220" H 6430 1550 20  0001 C CNN
+F 2 "local_libraries:TO_220_heatsink" H 6430 1550 20  0001 C CNN
 F 3 "" H 6400 1400 60  0001 C CNN
 	1    6400 1400
