File: hardware/kicad/v1_0/arduino_nano_reflow_TRIAC_v1_0.sch (KiCad schematic (older format))
At the start: 30 parts, among them J1 AC IN 220v, J10 CONN_01X17, J11 CONN_01X03, J12 MOUNTING_HOLE, J13 MOUNTING_HOLE, J14 MOUNTING_HOLE, J15 MOUNTING_HOLE, J2 HEATER, J3 DC IN 12V, J4 12V FAN, J9 CONN_01X05, Q1 IRF540N, U1 MOC3020M

Commit message: update - poslane do vyroby
Parts:
- removed J10: CONN_01X17, Connector_PinHeader_2.54mm:PinHeader_1x17_P2.54mm_Vertical, symbol Connector_Generic:Conn_01x17
- removed J15: MOUNTING_HOLE, MountingHole:MountingHole_3.2mm_M3_Pad, symbol arduino_nano_reflow_TRIAC_v1_0-rescue:CONN_01X01
- added C3: 100n, Capacitor_SMD:C_0805_2012Metric, symbol Device:C
- added J5: CONN_01X04, Connector_PinHeader_2.54mm:PinHeader_1x04_P2.54mm_Vertical, symbol Connector_Generic:Conn_01x04
- added J6: K-thermocouple, TerminalBlock_Phoenix:TerminalBlock_Phoenix_MKDS-1,5-2_1x02_P5.00mm_Horizontal, symbol arduino_nano_reflow_TRIAC_v1_0-rescue:Screw_Terminal_1x02
- added U2: MAX6675, Package_SO:SO-8_3.9x4.9mm_P1.27mm, symbol max6675:MAX6675
- J9: value CONN_01X05 -> MAX6675
Connections:
- net 5V: now also C3.2, J5.2 (Pin_2), U2.4 (VCC)
- net GND: now also C3.1, J5.1 (Pin_1), J6.2, U2.1 (GND), U2.2 (T-)
- net MISO: now also U2.7 (SO)
- net SCK: now also U2.5 (SCK)
- net TC_CS: now also U2.6 (CS)
- net D4 renamed SEGMENT_DIO
- net SEGMENT_DIO: now also J5.3 (Pin_3)
- net D5 renamed SEGMENT_CLK
- net SEGMENT_CLK: now also J5.4 (Pin_4)
- new net: J6.1, U2.3 (T+)
Other:
- note added: "Either use J9 or U2"
- note added: "TM1637 display header"
- moved on the sheet: F1
Changed lines of the file:
@@
 	0    1    -1   0
 $EndComp
-Text Label 9800 3650 0    47   ~ 0
-LCD_CS
-Text Label 9800 3550 0    47   ~ 0
-LCD_DC
-Text Label 9800 3450 0    47   ~ 0
-LCD_RESET
 Text Label 9800 2100 0    47   ~ 0
 MISO
-Text Label 9800 3950 0    47   ~ 0
-MISO
-Text Label 9950 3850 0    47   ~ 0
-MOSI
-Text Label 9800 3350 0    47   ~ 0
-SD_CS
 Text Label 1400 1850 2    47   ~ 0
 ZEROX
@@
 NoConn ~ 3200 4050
 NoConn ~ 3200 4250
-NoConn ~ 3200 4350
 NoConn ~ 1700 1750
 $Comp
@@
 Text GLabel 7150 4500 1    60   Input ~ 0
 12v
-Text GLabel 10000 2500 2    60   Input ~ 0
+Text GLabel 8825 2100 2    60   Input ~ 0
 GND
 Text GLabel 5850 3550 0    60   Input ~ 0
@@
 Text GLabel 2100 4150 0    60   Input ~ 0
 GND
-Text GLabel 9950 4550 2    60   Input ~ 0
-GND
 Text Label 9800 2200 0    47   ~ 0
 TC_CS
-Text Label 9800 3050 0    47   ~ 0
-D4
-Text Label 9800 3150 0    47   ~ 0
-D5
-Text Label 9800 3250 0    47   ~ 0
-D6
 $Comp
 L Transistor_FET:IRF540N Q1
@@
 P 9600 2300
 F 0 "J9" H 9600 2600 50  0000 C CNN
-F 1 "CONN_01X05" V 9700 2300 50  0000 C CNN
+F 1 "MAX6675" V 9700 2300 50  0000 C CNN
 F 2 "Connector_PinHeader_2.54mm:PinHeader_1x05_P2.54mm_Vertical" H 9600 2300 50  0001 C CNN
 F 3 "" H 9600 2300 50  0001 C CNN
@@
 Text Label 3200 3850 0    60   ~ 0
 VIN
-$Comp
-L Connector_Generic:Conn_01x17 J10
-U 1 1 592F1E66
-P 9600 3750
-F 0 "J10" H 9600 4650 50  0000 C CNN
-F 1 "CONN_01X17" V 9700 3750 50  0000 C CNN
-F 2 "Connector_PinHeader_2.54mm:PinHeader_1x17_P2.54mm_Vertical" H 9600 3750 50  0001 C CNN
-F 3 "" H 9600 3750 50  0001 C CNN
-	1    9600 3750
-	-1   0    0    1
-$EndComp
-Text GLabel 10000 2950 2    60   Input ~ 0
-GND
 Text GLabel 9800 2400 2    60   Input ~ 0
 5V
@@
 MOC_AC1
 $Comp
-L arduino_nano_reflow_TRIAC_v1_0-rescue:CONN_01X01 J15
-U 1 1 59493D8A
-P 2650 6950
-F 0 "J15" H 2650 7050 50  0000 C CNN
-F 1 "MOUNTING_HOLE" H 3100 6950 50  0000 C CNN
-F 2 "MountingHole:MountingHole_3.2mm_M3_Pad" H 2650 6950 50  0001 C CNN
-F 3 "" H 2650 6950 50  0001 C CNN
-	1    2650 6950
-	1    0    0    -1
-$EndComp
-$Comp
 L arduino_nano_reflow_TRIAC_v1_0-rescue:CONN_01X01 J12
 U 1 1 59493E77
@@
 Text GLabel 4400 3950 2    60   Input ~ 0
 GND
-Text Label 2350 4450 2    47   ~ 0
-D4
-Text Label 2350 4550 2    47   ~ 0
-D5
 Text Label 2350 4650 2    47   ~ 0
 D6
@@
 Wire Wire Line
 	6850 5150 6900 5150
-Wire Wire Line
-	10000 2950 9800 2950
-Wire Wire Line
-	9800 3850 9950 3850
-Wire Wire Line
-	9800 3750 9800 3850
-Wire Wire Line
-	9800 4150 9950 4150
-Wire Wire Line
-	9800 4050 9800 4150
-Wire Wire Line
-	9800 4550 9950 4550
-Wire Wire Line
-	9800 4450 9800 4550
-Wire Wire Line
-	9800 4350 9950 4350
-Wire Wire Line
-	9800 4250 9800 4350
 Wire Wire Line
 	1550 2050 1700 2050
@@
 Text GLabel 4400 2550 0    60   Input ~ 0
 AC1_OUT
-Text Label 9950 4150 0    47   ~ 0
-SCK
 Wire Notes Line
 	5050 3400 1050 3400
@@
 Wire Wire Line
 	10000 2500 9800 2500
-Text GLabel 9950 4350 2    60   Input ~ 0
-5V
 $Comp
 L Device:Fuse F1
 U 1 1 59639C08
-P 8800 5150
-F 0 "F1" H 8880 5150 50  0000 C CNN
-F 1 "Fuse" V 8725 5150 50  0000 C CNN
-F 2 "Fuse_Holders_and_Fuses:Fuseholder5x20_horiz_open_inline_Type-I" V 8730 5150 50  0001 C CNN
-F 3 "" H 8800 5150 50  0001 C CNN
-	1    8800 5150
+P 7450 6100
+F 0 "F1" H 7530 6100 50  0000 C CNN
+F 1 "Fuse" V 7375 6100 50  0000 C CNN
+F 2 "Fuse_Holders_and_Fuses:Fuseholder5x20_horiz_open_inline_Type-I" V 7380 6100 50  0001 C CNN
+F 3 "" H 7450 6100 50  0001 C CNN
+	1    7450 6100
 	0    1    1    0
 $EndComp
-Text GLabel 8650 5150 0    60   Input ~ 0
+Text GLabel 7300 6100 0    60   Input ~ 0
 AC2_IN
-Text GLabel 8950 5150 2    60   Input ~ 0
+Text GLabel 7600 6100 2    60   Input ~ 0
 AC2_OUT
 Wire Wire Line
@@
 Wire Wire Line
 	2275 6950 2275 7000
-Wire Wire Line
-	2450 6950 2275 6950
 Wire Wire Line
 	2450 6600 2275 6600
@@
 	0    -1   -1   0
 $EndComp
+$Comp
+L Connector_Generic:Conn_01x04 J5
+U 1 1 5FFCE5E8
+P 8275 2200
+F 0 "J5" H 8275 2400 50  0000 C CNN
+F 1 "CONN_01X04" V 8375 2200 50  0000 C CNN
+F 2 "Connector_PinHeader_2.54mm:PinHeader_1x04_P2.54mm_Vertical" H 8275 2200 50  0001 C CNN
+F 3 "" H 8275 2200 50  0001 C CNN
+	1    8275 2200
+	-1   0    0    -1
+$EndComp
+Text Notes 7850 1875 0    60   ~ 0
+TM1637 display header
+Text GLabel 9075 2200 2    60   Input ~ 0
+5V
+Text Label 8475 2300 0    60   ~ 0
+SEGMENT_DIO
+Wire Wire Line
+	8475 2200 9075 2200
+Wire Wire Line
+	8475 2100 8825 2100
+Text Label 8475 2400 0    60   ~ 0
+SEGMENT_CLK
+Text Label 2350 4450 2    60   ~ 0
+SEGMENT_DIO
+Text Label 2350 4550 2    60   ~ 0
+SEGMENT_CLK
+Text GLabel 10000 2500 2    60   Input ~ 0
+GND
+$Comp
+L arduino_nano_reflow_TRIAC_v1_0-rescue:Screw_Terminal_1x02 J6
+U 1 1 60037353
+P 10000 4525
+F 0 "J6" H 10000 4775 50  0000 C TNN
+F 1 "K-thermocouple" V 9850 4525 50  0000 C TNN
+F 2 "TerminalBlock_Phoenix:TerminalBlock_Phoenix_MKDS-1,5-2_1x02_P5.00mm_Horizontal" H 10000 4300 50  0001 C CNN
+F 3 "" H 9975 4525 50  0001 C CNN
+	1    10000 4525
+	-1   0    0    -1
+$EndComp
+Text GLabel 8925 3625 1    60   Input ~ 0
+5V
+Text GLabel 9525 5350 3    60   Input ~ 0
+GND
+$Comp
+L max6675:MAX6675 U2
+U 1 1 6004A91B
+P 8825 4725
+F 0 "U2" H 8875 4325 60  0000 C CNN
+F 1 "MAX6675" H 9025 4425 60  0000 C CNN
+F 2 "Package_SO:SO-8_3.9x4.9mm_P1.27mm" H 8875 4725 60  0001 C CNN
+F 3 "" H 8825 4725 60  0000 C CNN
+	1    8825 4725
+	1    0    0    -1
+$EndComp
+NoConn ~ 3200 4350
+Wire Wire Line
+	8675 5125 8675 5250
+Wire Wire Line
+	8675 5250 9525 5250
+Wire Wire Line
+	9525 5250 9525 4625
+Wire Wire Line
+	9525 4625 9375 4625
+Wire Wire Line
+	9525 4625 9800 4625
+Connection ~ 9525 4625
+Wire Wire Line
+	9525 5250 9525 5350
+Connection ~ 9525 5250
+Wire Wire Line
+	9375 4475 9650 4475
+Wire Wire Line
+	9650 4475 9650 4425
+Wire Wire Line
+	9650 4425 9800 4425
+$Comp
+L Device:C C3
+U 1 1 6006EEE2
+P 9475 3800
+F 0 "C3" V 9350 3725 70  0000 L BNN
+F 1 "100n" V 9675 3675 70  0000 L BNN
+F 2 "Capacitor_SMD:C_0805_2012Metric" H 9465 3590 65  0001 L TNN
+F 3 "" H 9475 3800 60  0001 C CNN
+	1    9475 3800
+	0    1    1    0
+$EndComp
+Wire Wire Line
+	8925 3975 8925 3800
+Wire Wire Line
+	9325 3800 8925 3800
+Connection ~ 8925 3800
+Wire Wire Line
+	8925 3800 8925 3625
+Text GLabel 9700 3800 2    60   Input ~ 0
+GND
+Wire Wire Line
+	9625 3800 9700 3800
+Text Label 8425 4275 2    47   ~ 0
+TC_CS
+Text Label 8425 4425 2    47   ~ 0
+SCK
+Text Label 8425 4575 2    47   ~ 0
+MISO
+Text Notes 8650 3175 0    60   ~ 0
+Either use J9 or U2
 $EndSCHEMATC
